Commit message: Add head/tail teleop control and fix limping gait
Adds W/A/S/D head pan/tilt and space-stepped tail control, each driven by
its own ros2_control position controller. Fixes the visible limp that
appeared once head/tail became actuated: Fast DDS's shared-memory transport
silently drops /cmd_vel on this machine, tripping the gait watchdog
mid-stride, so the project now runs on Cyclone DDS. Also rebalances body
mass to recover the trunk pitch inertia that moved off fixed joints and
onto the newly free head/tail bodies.

File: src/robot_cat_description/urdf/cat.ros2_control.xacro (robot description, xacro)
@@ -32,4 +32,7 @@
       <xacro:leg_control prefix="rl"/>
       <xacro:leg_control prefix="rr"/>
+      <xacro:joint_control name="neck_pan_joint"/>
+      <xacro:joint_control name="head_tilt_joint"/>
+      <xacro:joint_control name="tail_joint"/>
     </ros2_control>
     <gazebo>

File: src/robot_cat_description/urdf/cat.urdf.xacro (robot description, xacro)
@@ -20,6 +20,23 @@
   <xacro:property name="hip_x" value="0.11"/>
   <xacro:property name="hip_y" value="0.055"/>
-  <!-- ==================== masses ==================== -->
-  <xacro:property name="body_mass"  value="2.0"/>
+  <!-- ==================== masses ====================
+       The head and tail are cosmetic but no longer fixed joints, so their
+       mass is a free body hanging off the trunk instead of being lumped into
+       it by SDF conversion. Two things follow, and both showed up as a
+       visibly bouncier trot when the tail was actuated:
+       * the trunk lost the parallel-axis share those masses used to
+         contribute to its pitch inertia (0.0263 -> 0.0164, a 38% drop), so
+         it now pitches far more readily each half stride;
+       * whatever mass they keep slops about on a long lever at the very
+         ends of the body, exactly where it disturbs pitch most.
+       So they carry token mass, damped enough to settle rather than swing,
+       and `body_mass` carries what they gave up - total mass is unchanged. -->
+  <xacro:property name="body_mass"  value="2.23"/>
+  <xacro:property name="head_mass"  value="0.06"/>
+  <xacro:property name="neck_mass"  value="0.01"/>
+  <xacro:property name="tail_mass"  value="0.015"/>
+  <!-- Cosmetic joints only. Far stiffer than the legs: they are meant to hold
+       a pose, and any wobble here feeds straight back into the trunk. -->
+  <xacro:property name="trim_damping" value="0.4"/>
   <xacro:property name="hip_mass"   value="0.10"/>
   <xacro:property name="thigh_mass" value="0.12"/>
@@ -56,10 +73,31 @@
     <xacro:box_inertia mass="${body_mass}" x="${body_length}" y="${body_width}" z="${body_height}"/>
   </link>
-  <!-- Cosmetic head and tail. Fixed joints, so SDF conversion folds their mass
-       into base_link; they exist to make orientation obvious on screen. -->
-  <joint name="head_joint" type="fixed">
+  <!-- Head: two actuated DOF (pan, tilt) driven by head_position_controller
+       from the W/A/S/D keys - see robot_cat_teleop/head.py. neck_link is a
+       near-massless intermediate body so pan and tilt are independent
+       revolute joints rather than one compound one; ros2_control needs each
+       DOF as its own joint. -->
+  <joint name="neck_pan_joint" type="revolute">
     <parent link="base_link"/>
+    <child link="neck_link"/>
+    <origin xyz="${body_length/2} 0 ${body_height/2}" rpy="0 0 0"/>
+    <axis xyz="0 0 1"/>
+    <limit lower="-0.6" upper="0.6" effort="5" velocity="6"/>
+    <dynamics damping="${trim_damping}" friction="${joint_friction}"/>
+  </joint>
+  <link name="neck_link">
+    <xacro:box_inertia mass="${neck_mass}" x="0.02" y="0.02" z="0.02"/>
+  </link>
+  <joint name="head_tilt_joint" type="revolute">
+    <parent link="neck_link"/>
     <child link="head_link"/>
-    <origin xyz="${body_length/2 + 0.03} 0 ${body_height/2}" rpy="0 0 0"/>
+    <origin xyz="0.03 0 0" rpy="0 0 0"/>
+    <!-- Axis is -Y, not +Y: with the head extending along local +X, a
+         positive rotation about +Y points the nose down, which is backwards
+         from "positive tilt = look up" used by the tilt_lower/tilt_upper
+         convention below and by robot_cat_teleop. -->
+    <axis xyz="0 -1 0"/>
+    <limit lower="-0.3" upper="0.5" effort="5" velocity="6"/>
+    <dynamics damping="${trim_damping}" friction="${joint_friction}"/>
   </joint>
   <link name="head_link">
@@ -84,10 +122,19 @@
       <material name="cat_accent"/>
     </visual>
-    <xacro:box_inertia mass="0.25" x="0.1" y="0.1" z="0.1"/>
+    <xacro:box_inertia mass="${head_mass}" x="0.1" y="0.1" z="0.1"/>
   </link>
-  <joint name="tail_joint" type="fixed">
+  <!-- Tail: one actuated DOF, stepped by the space bar - see
+       robot_cat_teleop/tail.py. The -0.9 rad pitch in the origin is the rest
+       pose, tail up and back; the joint angle is measured from there, so
+       positive raises towards vertical and negative droops it down. -->
+  <joint name="tail_joint" type="revolute">
     <parent link="base_link"/>
     <child link="tail_link"/>
     <origin xyz="${-body_length/2 - 0.04} 0 ${body_height/2}" rpy="0 -0.9 0"/>
+    <axis xyz="0 1 0"/>
+    <!-- Wider than the sweep TailParams actually uses, so the controller
+         settles on its target instead of pushing against the joint stop. -->
+    <limit lower="-1.4" upper="1.0" effort="5" velocity="6"/>
+    <dynamics damping="${trim_damping}" friction="${joint_friction}"/>
   </joint>
   <link name="tail_link">
@@ -97,5 +144,5 @@
       <material name="cat_accent"/>
     </visual>
-    <xacro:cylinder_inertia mass="0.05" radius="0.009" length="0.12"/>
+    <xacro:cylinder_inertia mass="${tail_mass}" radius="0.009" length="0.12"/>
   </link>
   <!-- ==================== legs ====================
