Commit message: Give the cat eyes, and a meow on the m key
The eyes are cosmetic but sited where a stereo pair would really go, so
camera sensors can be mounted at the same origins once perception moves to
Linux - Gazebo cannot run camera sensors on macOS at all (gz-sim#960).

The meow plays through the host rather than the simulation, because Gazebo
has no audio component of any kind. The clip is synthesised from a harmonic
stack under a swept formant filter rather than sampled, which keeps the repo
self-contained and free of any sample licence, and it is rate-limited: key
autorepeat would otherwise spawn a player process per repeat.

File: src/robot_cat_description/urdf/cat.urdf.xacro (robot description, xacro)
@@ -62,4 +62,6 @@
   <material name="cat_paw">    <color rgba="0.15 0.15 0.15 1.0"/></material>
   <material name="cat_nose">   <color rgba="0.85 0.55 0.60 1.0"/></material>
+  <material name="cat_eye">    <color rgba="0.92 0.90 0.55 1.0"/></material>
+  <material name="cat_pupil">  <color rgba="0.05 0.05 0.05 1.0"/></material>
   <!-- ==================== body ==================== -->
   <link name="base_link">
@@ -111,4 +113,29 @@
       <material name="cat_nose"/>
     </visual>
+    <!-- Eyes. Cosmetic for now, but placed where a stereo pair would actually
+         go: forward-facing on the head sphere, level, and separated by
+         2*eye_y. When perception moves to Linux, mount the camera sensors at
+         these same origins and the view will match what you see here. Gazebo
+         cannot run camera sensors on macOS at all - Cocoa requires render
+         window creation on the main thread (gazebosim/gz-sim#960). -->
+    <xacro:property name="eye_x" value="0.036"/>
+    <xacro:property name="eye_y" value="0.022"/>
+    <xacro:property name="eye_z" value="0.018"/>
+    <xacro:macro name="cat_eye" params="side y_sign">
+      <visual name="eye_${side}">
+        <origin xyz="${eye_x} ${y_sign * eye_y} ${eye_z}" rpy="0 0 0"/>
+        <geometry><sphere radius="0.010"/></geometry>
+        <material name="cat_eye"/>
+      </visual>
+      <visual name="pupil_${side}">
+        <!-- Sits just proud of the eyeball so it renders in front of it
+             rather than z-fighting with the white. -->
+        <origin xyz="${eye_x + 0.007} ${y_sign * eye_y} ${eye_z}" rpy="0 0 0"/>
+        <geometry><sphere radius="0.005"/></geometry>
+        <material name="cat_pupil"/>
+      </visual>
+    </xacro:macro>
+    <xacro:cat_eye side="left"  y_sign="1"/>
+    <xacro:cat_eye side="right" y_sign="-1"/>
     <!-- ears -->
     <visual>

Commit message: Mirror the rear legs' knee so the cat is anatomically right
Every leg used the front-leg calf range and IK branch, so all four bent the
same way. A real quadruped's hind knee bends toward the head while the front
elbow bends toward the tail, and the uniform version read as wrong on sight
without being easy to name.

leg.xacro now takes a knee_sign and mirrors the calf joint's own limit range
for the rear pair; gait.py derives the matching IK sign per leg. The two must
agree or the IK solves for a branch the joint cannot physically reach.

Foot placement is unchanged - knee_sign only picks which of the two IK
solutions reaches a given target - so the gait is untouched. Verified in
Gazebo: 1.99 m in 12 s with 1.2 deg of heading drift, no worse than before.

thigh_lower goes -1.20 -> -1.45: the mirrored knee needs the thigh to swing
further negative to reach poses the front leg reaches by swinging positive,
and the full lie-down fold wanted -1.318, which -1.20 clipped.

File: src/robot_cat_description/urdf/cat.urdf.xacro (robot description, xacro)
@@ -47,5 +47,10 @@
        the IK branch (knee_sign = -1 in leg_ik.py). -->
   <xacro:property name="hip_range"      value="0.80"/>
-  <xacro:property name="thigh_lower"    value="-1.20"/>
+  <!-- -1.20 was enough when every leg used the same front-elbow-style knee
+       branch: the rear legs' full lie-down fold now needs the mirrored
+       branch's thigh to swing to -1.318 rad, and -1.20 clipped it by 0.12
+       rad. -1.45 leaves margin over that, the same way down_stance_height in
+       lie_down.py leaves margin over the calf stop rather than sitting on it. -->
+  <xacro:property name="thigh_lower"    value="-1.45"/>
   <xacro:property name="thigh_upper"    value="2.60"/>
   <xacro:property name="calf_lower"     value="-2.70"/>
@@ -176,8 +181,12 @@
        Joint order fl, fr, rl, rr is the contract with the gait node and
        controllers.yaml. Do not reorder without changing both. -->
-  <xacro:cat_leg prefix="fl" x_sign="1"  y_sign="1"/>
-  <xacro:cat_leg prefix="fr" x_sign="1"  y_sign="-1"/>
-  <xacro:cat_leg prefix="rl" x_sign="-1" y_sign="1"/>
-  <xacro:cat_leg prefix="rr" x_sign="-1" y_sign="-1"/>
+  <!-- knee_sign picks which way the calf joint's own limit range points -
+       see the comment on it in leg.xacro for why this exists at all: a real
+       quadruped's hind knee bends the opposite way from its front elbow, and
+       without this every leg looked like a front leg. -->
+  <xacro:cat_leg prefix="fl" x_sign="1"  y_sign="1"  knee_sign="-1"/>
+  <xacro:cat_leg prefix="fr" x_sign="1"  y_sign="-1" knee_sign="-1"/>
+  <xacro:cat_leg prefix="rl" x_sign="-1" y_sign="1"  knee_sign="1"/>
+  <xacro:cat_leg prefix="rr" x_sign="-1" y_sign="-1" knee_sign="1"/>
   <gazebo reference="base_link">
     <material>Gazebo/Grey</material>

File: src/robot_cat_description/urdf/leg.xacro (robot description, xacro)
@@ -6,8 +6,21 @@
        robot_cat_gait/leg_ik.py. The gait solver assumes exactly this chain and
        these axes.
-       prefix  - leg name, one of fl / fr / rl / rr
-       x_sign  - +1 front, -1 rear
-       y_sign  - +1 left,  -1 right -->
-  <xacro:macro name="cat_leg" params="prefix x_sign y_sign">
+       prefix     - leg name, one of fl / fr / rl / rr
+       x_sign     - +1 front, -1 rear
+       y_sign     - +1 left,  -1 right
+       knee_sign  - which of the two IK elbow solutions the calf joint's own
+                    range points at: -1 for front (elbow bends toward the
+                    tail, like a real front leg), +1 for rear (knee bends
+                    toward the head, like a real hind leg). Every real
+                    quadruped's hind knee bends the opposite way from its
+                    front elbow; giving all four legs the same calf range
+                    made the rear legs look like front legs grafted on
+                    backwards - anatomically wrong, and it reads as wrong on
+                    sight even without a name for why.
+                    This must match GaitGenerator's per-leg knee sign in
+                    gait.py (derived the same way, from x_sign), or the IK
+                    solves for a branch the joint cannot physically reach and
+                    the leg locks against its own stop. -->
+  <xacro:macro name="cat_leg" params="prefix x_sign y_sign knee_sign">
     <!-- hip: abduction / adduction -->
     <joint name="${prefix}_hip_joint" type="revolute">
@@ -59,5 +72,9 @@
       <origin xyz="0 0 ${-thigh_length}" rpy="0 0 0"/>
       <axis xyz="0 1 0"/>
-      <limit lower="${calf_lower}" upper="${calf_upper}"
+      <!-- Mirrored for knee_sign > 0: same range width, reflected through
+           zero, so a rear leg's calf can only reach the positive angles its
+           forward-bending IK branch actually produces. -->
+      <limit lower="${calf_lower if knee_sign &lt; 0 else -calf_upper}"
+             upper="${calf_upper if knee_sign &lt; 0 else -calf_lower}"
              effort="${joint_effort}" velocity="${joint_velocity}"/>
       <dynamics damping="${joint_damping}" friction="${joint_friction}"/>
