Commit message: Give all four legs the same knee, as real quadruped robots have
Reverts 1559b06, which mirrored the rear calf range and IK branch so the hind
knees bent toward the head the way a real cat's do. That was correct anatomy,
but it is not how machines of this class are built: Spot, Unitree and the rest
put four identical legs on the corners, and matching them is the look we want
here.

Mechanically this is the pre-1559b06 arrangement restored in full. knee_sign
survives as the IK branch selector but is one value for the whole robot again,
so leg.xacro no longer takes it per leg and gait.py no longer derives it from
which end of the body a leg is on.

thigh_lower goes back -1.45 -> -1.20. The wider range only ever existed because
a mirrored rear knee needed the thigh to swing further negative to reach the
full lie-down fold; with uniform legs the fold sits inside -1.20 again, which
the joint-limit tests cover for stretch and lie-down alike.

Test count 579 -> 573: the six assertions that pinned the mirroring go with it.

Co-Authored-By: Claude Opus 5 <noreply@anthropic.com>

File: src/robot_cat_description/urdf/cat.urdf.xacro (robot description, xacro)
@@ -47,10 +47,5 @@
        the IK branch (knee_sign = -1 in leg_ik.py). -->
   <xacro:property name="hip_range"      value="0.80"/>
-  <!-- -1.20 was enough when every leg used the same front-elbow-style knee
-       branch: the rear legs' full lie-down fold now needs the mirrored
-       branch's thigh to swing to -1.318 rad, and -1.20 clipped it by 0.12
-       rad. -1.45 leaves margin over that, the same way down_stance_height in
-       lie_down.py leaves margin over the calf stop rather than sitting on it. -->
-  <xacro:property name="thigh_lower"    value="-1.45"/>
+  <xacro:property name="thigh_lower"    value="-1.20"/>
   <xacro:property name="thigh_upper"    value="2.60"/>
   <xacro:property name="calf_lower"     value="-2.70"/>
@@ -181,12 +176,8 @@
        Joint order fl, fr, rl, rr is the contract with the gait node and
        controllers.yaml. Do not reorder without changing both. -->
-  <!-- knee_sign picks which way the calf joint's own limit range points -
-       see the comment on it in leg.xacro for why this exists at all: a real
-       quadruped's hind knee bends the opposite way from its front elbow, and
-       without this every leg looked like a front leg. -->
-  <xacro:cat_leg prefix="fl" x_sign="1"  y_sign="1"  knee_sign="-1"/>
-  <xacro:cat_leg prefix="fr" x_sign="1"  y_sign="-1" knee_sign="-1"/>
-  <xacro:cat_leg prefix="rl" x_sign="-1" y_sign="1"  knee_sign="1"/>
-  <xacro:cat_leg prefix="rr" x_sign="-1" y_sign="-1" knee_sign="1"/>
+  <xacro:cat_leg prefix="fl" x_sign="1"  y_sign="1"/>
+  <xacro:cat_leg prefix="fr" x_sign="1"  y_sign="-1"/>
+  <xacro:cat_leg prefix="rl" x_sign="-1" y_sign="1"/>
+  <xacro:cat_leg prefix="rr" x_sign="-1" y_sign="-1"/>
   <gazebo reference="base_link">
     <material>Gazebo/Grey</material>

File: src/robot_cat_description/urdf/leg.xacro (robot description, xacro)
@@ -6,21 +6,8 @@
        robot_cat_gait/leg_ik.py. The gait solver assumes exactly this chain and
        these axes.
-       prefix     - leg name, one of fl / fr / rl / rr
-       x_sign     - +1 front, -1 rear
-       y_sign     - +1 left,  -1 right
-       knee_sign  - which of the two IK elbow solutions the calf joint's own
-                    range points at: -1 for front (elbow bends toward the
-                    tail, like a real front leg), +1 for rear (knee bends
-                    toward the head, like a real hind leg). Every real
-                    quadruped's hind knee bends the opposite way from its
-                    front elbow; giving all four legs the same calf range
-                    made the rear legs look like front legs grafted on
-                    backwards - anatomically wrong, and it reads as wrong on
-                    sight even without a name for why.
-                    This must match GaitGenerator's per-leg knee sign in
-                    gait.py (derived the same way, from x_sign), or the IK
-                    solves for a branch the joint cannot physically reach and
-                    the leg locks against its own stop. -->
-  <xacro:macro name="cat_leg" params="prefix x_sign y_sign knee_sign">
+       prefix  - leg name, one of fl / fr / rl / rr
+       x_sign  - +1 front, -1 rear
+       y_sign  - +1 left,  -1 right -->
+  <xacro:macro name="cat_leg" params="prefix x_sign y_sign">
     <!-- hip: abduction / adduction -->
     <joint name="${prefix}_hip_joint" type="revolute">
@@ -72,9 +59,5 @@
       <origin xyz="0 0 ${-thigh_length}" rpy="0 0 0"/>
       <axis xyz="0 1 0"/>
-      <!-- Mirrored for knee_sign > 0: same range width, reflected through
-           zero, so a rear leg's calf can only reach the positive angles its
-           forward-bending IK branch actually produces. -->
-      <limit lower="${calf_lower if knee_sign &lt; 0 else -calf_upper}"
-             upper="${calf_upper if knee_sign &lt; 0 else -calf_lower}"
+      <limit lower="${calf_lower}" upper="${calf_upper}"
              effort="${joint_effort}" velocity="${joint_velocity}"/>
       <dynamics damping="${joint_damping}" friction="${joint_friction}"/>

Commit message: Stand the cat on cat-proportioned legs instead of dachshund ones
The silhouette was wrong in a way that measures: 18.7 cm at the withers over a
22 cm hip span, a ratio of 0.85. A cat is close to square in profile - about as
tall at the shoulder as its trunk is long, roughly 24 cm at the withers on a
real animal - so 0.85 read as a long, low body on short legs.

Segments go 0.09 -> 0.11 and stance_height 0.13 -> 0.16, which puts the withers
at 21.7 cm for a ratio of 0.99.

Those two had to move together. What the gait depends on is not the absolute
height but how far the knee stays bent, and the old leg stood at 73% of full
reach. Raising stance_height alone would have taken that to 91% - a nearly
locked leg with no room left to swing or absorb a landing. At 0.11 segments,
0.16 holds the same 73%.

Link masses scale with the lengthening (0.12 -> 0.147, 0.08 -> 0.098) so the
longer links do not quietly become less dense than the ones they replace.

Measured in cat_world after the change, against the same walk before it:

    forward speed   0.170 m/s   (was 0.17)
    body roll p-p   2.9 deg     (was 2.9)
    heading drift   1.6 deg over 3.2 m
    standing height 0.171999    (predicted 0.172)

So the taller stance costs nothing: the higher centre of mass did not eat into
the roll stiffness stance_width bought, and the joint-limit tests pass for the
stretch and lie-down poses unchanged.

Note the lengths are declared in three places, not two - cat.urdf.xacro,
LegGeometry in leg_ik.py, and the parameter defaults in gait_controller.py.

Co-Authored-By: Claude Opus 5 <noreply@anthropic.com>

File: src/robot_cat_description/urdf/cat.urdf.xacro (robot description, xacro)
@@ -11,6 +11,12 @@
        places the legs cannot reach. -->
   <xacro:property name="hip_offset"   value="0.035"/>  <!-- hip roll -> thigh pitch, lateral -->
-  <xacro:property name="thigh_length" value="0.09"/>   <!-- L1 -->
-  <xacro:property name="calf_length"  value="0.09"/>   <!-- L2 -->
+  <!-- 0.09 made a long, low animal: 18.7 cm at the withers over a 22 cm hip
+       span, a ratio of 0.85. A cat is close to square in profile - it stands
+       about as tall at the shoulder as its trunk is long - so the old figure
+       read as a dachshund. 0.11 puts the withers at 21.7 cm for a ratio of
+       0.99, and holds the standing knee at the same 73% of full reach the
+       0.09 leg had, so the gait keeps its bend and its swing clearance. -->
+  <xacro:property name="thigh_length" value="0.11"/>   <!-- L1 -->
+  <xacro:property name="calf_length"  value="0.11"/>   <!-- L2 -->
   <xacro:property name="foot_radius"  value="0.012"/>
   <xacro:property name="body_length" value="0.30"/>
@@ -40,6 +46,8 @@
   <xacro:property name="trim_damping" value="0.4"/>
   <xacro:property name="hip_mass"   value="0.10"/>
-  <xacro:property name="thigh_mass" value="0.12"/>
-  <xacro:property name="calf_mass"  value="0.08"/>
+  <!-- Scaled with the 0.09 -> 0.11 lengthening, so the longer links do not
+       quietly become less dense than the ones they replaced. -->
+  <xacro:property name="thigh_mass" value="0.147"/>
+  <xacro:property name="calf_mass"  value="0.098"/>
   <!-- ==================== joint properties ====================
        Ranges are deliberately generous for the pitch joints so the gait has

Commit message: Make body size one knob, and give the trunk a cat's cross-section
Two changes, both driven by the brief ("ok. 50 centymetrów wysokości i
przypominał kota") which the model was missing in two different ways.

Size is now a single parameter threaded through the model and the gait
together, so it can be chosen by measurement instead of assumed:

    ./run/docker/sim.sh scale:=1.87

Lengths go as scale, masses as scale^3 and joint effort as scale^4, which is
how joint torque actually scales - mass times lever arm. cycle_time is the one
exception and goes as sqrt(scale): a leg is a pendulum, so a bigger animal
swings it more slowly for the *same* gait. That is the Froude scaling that
makes a horse's walk and a cat's walk the same motion at different sizes.

At scale 1.87 the head reaches the 50 cm asked for. Measured there: 24.2 kg,
0.94 m/s, and 30.5 Nm at the 95th percentile against 3.4 Nm at scale 1.0. That
is a factor of nine from one line in a brief, and it rules out every servo on
the market - the fitted exponent is 3.5, lower than the 4 of pure mass x lever
only because the tempo is Froude-scaled.

Separately, the trunk was the wrong shape. A cat's chest is deeper than it is
wide - a girth of ~38 cm works out near 14 cm deep by 10 cm across - and the
box was 1 : 0.47 : 0.30 instead of 1 : 0.37 : 0.47. It read as a slab on legs.
hip_offset also comes in 0.035 -> 0.025 to stop the feet planting so far
outside the body.

Costs nothing: 0.943 m/s against 0.944 before, and body roll actually improves
from 1.6 to 1.4 degrees peak-to-peak. 581 tests pass.

The generated report is gitignored rather than tracked - it is rebuilt from
its script, and a binary that changes on every regeneration does not belong in
the history.

Co-Authored-By: Claude Opus 5 <noreply@anthropic.com>

File: src/robot_cat_description/urdf/cat.urdf.xacro (robot description, xacro)
@@ -6,9 +6,20 @@
   <xacro:arg name="use_gazebo" default="true"/>
   <xacro:arg name="controllers_file" default=""/>
+  <!-- ==================== scale ====================
+       One knob for the whole animal. Every length below is a base dimension
+       multiplied by this; masses go as scale^3 and joint effort as scale^4,
+       which is how joint torque actually scales (mass x lever arm).
+       1.00 is the 22 cm-at-the-withers cat the gait was tuned on, and 1.87
+       puts the head at the 50 cm the brief asks for. The second one is not a
+       cosmetic choice: the same scaling turns a 3.7 kg animal into a 24 kg
+       one whose joints need roughly 60 Nm, which rules out every servo and
+       most brushless actuators. Changing this picks an actuator class. -->
+  <xacro:arg name="scale" default="1.0"/>
+  <xacro:property name="scale" value="$(arg scale)"/>
   <!-- ==================== dimensions ====================
        These MUST match LegGeometry in robot_cat_gait/leg_ik.py. If you change
        a length here, change it there too, or the gait will command feet to
        places the legs cannot reach. -->
-  <xacro:property name="hip_offset"   value="0.035"/>  <!-- hip roll -> thigh pitch, lateral -->
+  <xacro:property name="hip_offset"   value="${0.025 * scale}"/>  <!-- hip roll -> thigh pitch, lateral -->
   <!-- 0.09 made a long, low animal: 18.7 cm at the withers over a 22 cm hip
        span, a ratio of 0.85. A cat is close to square in profile - it stands
@@ -17,13 +28,17 @@
        0.99, and holds the standing knee at the same 73% of full reach the
        0.09 leg had, so the gait keeps its bend and its swing clearance. -->
-  <xacro:property name="thigh_length" value="0.11"/>   <!-- L1 -->
-  <xacro:property name="calf_length"  value="0.11"/>   <!-- L2 -->
-  <xacro:property name="foot_radius"  value="0.012"/>
-  <xacro:property name="body_length" value="0.30"/>
-  <xacro:property name="body_width"  value="0.14"/>
-  <xacro:property name="body_height" value="0.09"/>
+  <xacro:property name="thigh_length" value="${0.11 * scale}"/>   <!-- L1 -->
+  <xacro:property name="calf_length"  value="${0.11 * scale}"/>   <!-- L2 -->
+  <xacro:property name="foot_radius"  value="${0.012 * scale}"/>
+  <!-- A cat's trunk is deeper than it is wide - chest girth of about
+       38 cm works out near 14 cm deep by 10 cm across - so the box is
+       length : width : depth = 1 : 0.37 : 0.47. The old 1 : 0.47 : 0.30 was
+       the other way round and read as a slab on legs rather than an animal. -->
+  <xacro:property name="body_length" value="${0.30 * scale}"/>
+  <xacro:property name="body_width"  value="${0.111 * scale}"/>
+  <xacro:property name="body_height" value="${0.141 * scale}"/>
   <!-- Hip joint placement relative to body centre. -->
-  <xacro:property name="hip_x" value="0.11"/>
-  <xacro:property name="hip_y" value="0.055"/>
+  <xacro:property name="hip_x" value="${0.11 * scale}"/>
+  <xacro:property name="hip_y" value="${0.055 * scale}"/>
   <!-- ==================== masses ====================
        The head and tail are cosmetic but no longer fixed joints, so their
@@ -38,16 +53,16 @@
        So they carry token mass, damped enough to settle rather than swing,
        and `body_mass` carries what they gave up - total mass is unchanged. -->
-  <xacro:property name="body_mass"  value="2.23"/>
-  <xacro:property name="head_mass"  value="0.06"/>
-  <xacro:property name="neck_mass"  value="0.01"/>
-  <xacro:property name="tail_mass"  value="0.015"/>
+  <xacro:property name="body_mass"  value="${2.23 * scale**3}"/>
+  <xacro:property name="head_mass"  value="${0.06 * scale**3}"/>
+  <xacro:property name="neck_mass"  value="${0.01 * scale**3}"/>
+  <xacro:property name="tail_mass"  value="${0.015 * scale**3}"/>
   <!-- Cosmetic joints only. Far stiffer than the legs: they are meant to hold
        a pose, and any wobble here feeds straight back into the trunk. -->
   <xacro:property name="trim_damping" value="0.4"/>
-  <xacro:property name="hip_mass"   value="0.10"/>
+  <xacro:property name="hip_mass"   value="${0.10 * scale**3}"/>
   <!-- Scaled with the 0.09 -> 0.11 lengthening, so the longer links do not
        quietly become less dense than the ones they replaced. -->
-  <xacro:property name="thigh_mass" value="0.147"/>
-  <xacro:property name="calf_mass"  value="0.098"/>
+  <xacro:property name="thigh_mass" value="${0.147 * scale**3}"/>
+  <xacro:property name="calf_mass"  value="${0.098 * scale**3}"/>
   <!-- ==================== joint properties ====================
        Ranges are deliberately generous for the pitch joints so the gait has
@@ -59,5 +74,5 @@
   <xacro:property name="calf_lower"     value="-2.70"/>
   <xacro:property name="calf_upper"     value="-0.10"/>
-  <xacro:property name="joint_effort"   value="20.0"/>
+  <xacro:property name="joint_effort"   value="${20.0 * scale**4}"/>
   <xacro:property name="joint_velocity" value="20.0"/>
   <xacro:property name="joint_damping"  value="0.05"/>
@@ -97,10 +112,10 @@
   </joint>
   <link name="neck_link">
-    <xacro:box_inertia mass="${neck_mass}" x="0.02" y="0.02" z="0.02"/>
+    <xacro:box_inertia mass="${neck_mass}" x="${0.02 * scale}" y="${0.02 * scale}" z="${0.02 * scale}"/>
   </link>
   <joint name="head_tilt_joint" type="revolute">
     <parent link="neck_link"/>
     <child link="head_link"/>
-    <origin xyz="0.03 0 0" rpy="0 0 0"/>
+    <origin xyz="${0.03 * scale} 0 0" rpy="0 0 0"/>
     <!-- Axis is -Y, not +Y: with the head extending along local +X, a
          positive rotation about +Y points the nose down, which is backwards
@@ -113,10 +128,10 @@
   <link name="head_link">
     <visual>
-      <geometry><sphere radius="0.05"/></geometry>
+      <geometry><sphere radius="${0.05 * scale}"/></geometry>
       <material name="cat_fur"/>
     </visual>
     <visual>
-      <origin xyz="0.045 0 0" rpy="0 0 0"/>
-      <geometry><sphere radius="0.012"/></geometry>
+      <origin xyz="${0.045 * scale} 0 0" rpy="0 0 0"/>
+      <geometry><sphere radius="${0.012 * scale}"/></geometry>
       <material name="cat_nose"/>
     </visual>
@@ -127,11 +142,11 @@
          cannot run camera sensors on macOS at all - Cocoa requires render
          window creation on the main thread (gazebosim/gz-sim#960). -->
-    <xacro:property name="eye_x" value="0.036"/>
-    <xacro:property name="eye_y" value="0.022"/>
-    <xacro:property name="eye_z" value="0.018"/>
+    <xacro:property name="eye_x" value="${0.036 * scale}"/>
+    <xacro:property name="eye_y" value="${0.022 * scale}"/>
+    <xacro:property name="eye_z" value="${0.018 * scale}"/>
     <xacro:macro name="cat_eye" params="side y_sign">
       <visual name="eye_${side}">
         <origin xyz="${eye_x} ${y_sign * eye_y} ${eye_z}" rpy="0 0 0"/>
-        <geometry><sphere radius="0.010"/></geometry>
+        <geometry><sphere radius="${0.010 * scale}"/></geometry>
         <material name="cat_eye"/>
       </visual>
@@ -139,6 +154,6 @@
         <!-- Sits just proud of the eyeball so it renders in front of it
              rather than z-fighting with the white. -->
-        <origin xyz="${eye_x + 0.007} ${y_sign * eye_y} ${eye_z}" rpy="0 0 0"/>
-        <geometry><sphere radius="0.005"/></geometry>
+        <origin xyz="${eye_x + 0.007 * scale} ${y_sign * eye_y} ${eye_z}" rpy="0 0 0"/>
+        <geometry><sphere radius="${0.005 * scale}"/></geometry>
         <material name="cat_pupil"/>
       </visual>
@@ -148,14 +163,14 @@
     <!-- ears -->
     <visual>
-      <origin xyz="-0.01 0.028 0.042" rpy="0 0 0"/>
-      <geometry><box size="0.02 0.012 0.035"/></geometry>
+      <origin xyz="${-0.01 * scale} ${0.028 * scale} ${0.042 * scale}" rpy="0 0 0"/>
+      <geometry><box size="${0.02 * scale} ${0.012 * scale} ${0.035 * scale}"/></geometry>
       <material name="cat_accent"/>
     </visual>
     <visual>
-      <origin xyz="-0.01 -0.028 0.042" rpy="0 0 0"/>
-      <geometry><box size="0.02 0.012 0.035"/></geometry>
+      <origin xyz="${-0.01 * scale} ${-0.028 * scale} ${0.042 * scale}" rpy="0 0 0"/>
+      <geometry><box size="${0.02 * scale} ${0.012 * scale} ${0.035 * scale}"/></geometry>
       <material name="cat_accent"/>
     </visual>
-    <xacro:box_inertia mass="${head_mass}" x="0.1" y="0.1" z="0.1"/>
+    <xacro:box_inertia mass="${head_mass}" x="${0.1 * scale}" y="${0.1 * scale}" z="${0.1 * scale}"/>
   </link>
   <!-- Tail: one actuated DOF, stepped by the space bar - see
@@ -166,5 +181,5 @@
     <parent link="base_link"/>
     <child link="tail_link"/>
-    <origin xyz="${-body_length/2 - 0.04} 0 ${body_height/2}" rpy="0 -0.9 0"/>
+    <origin xyz="${-body_length/2 - 0.04 * scale} 0 ${body_height/2}" rpy="0 -0.9 0"/>
     <axis xyz="0 1 0"/>
     <!-- Wider than the sweep TailParams actually uses, so the controller
@@ -175,9 +190,9 @@
   <link name="tail_link">
     <visual>
-      <origin xyz="0 0 0.04" rpy="0 0 0"/>
-      <geometry><cylinder radius="0.009" length="0.12"/></geometry>
+      <origin xyz="0 0 ${0.04 * scale}" rpy="0 0 0"/>
+      <geometry><cylinder radius="${0.009 * scale}" length="${0.12 * scale}"/></geometry>
       <material name="cat_accent"/>
     </visual>
-    <xacro:cylinder_inertia mass="${tail_mass}" radius="0.009" length="0.12"/>
+    <xacro:cylinder_inertia mass="${tail_mass}" radius="${0.009 * scale}" length="${0.12 * scale}"/>
   </link>
   <!-- ==================== legs ====================

File: src/robot_cat_description/urdf/leg.xacro (robot description, xacro)
@@ -23,8 +23,8 @@
       <visual>
         <origin xyz="0 ${y_sign * hip_offset / 2.0} 0" rpy="${pi/2} 0 0"/>
-        <geometry><cylinder radius="0.018" length="${hip_offset}"/></geometry>
+        <geometry><cylinder radius="${0.018 * scale}" length="${hip_offset}"/></geometry>
         <material name="cat_accent"/>
       </visual>
-      <xacro:cylinder_inertia mass="${hip_mass}" radius="0.018" length="${hip_offset}"/>
+      <xacro:cylinder_inertia mass="${hip_mass}" radius="${0.018 * scale}" length="${hip_offset}"/>
     </link>
     <!-- thigh: hip pitch -->
@@ -41,12 +41,12 @@
       <visual>
         <origin xyz="0 0 ${-thigh_length / 2.0}" rpy="0 0 0"/>
-        <geometry><cylinder radius="0.014" length="${thigh_length}"/></geometry>
+        <geometry><cylinder radius="${0.014 * scale}" length="${thigh_length}"/></geometry>
         <material name="cat_fur"/>
       </visual>
       <collision>
         <origin xyz="0 0 ${-thigh_length / 2.0}" rpy="0 0 0"/>
-        <geometry><cylinder radius="0.014" length="${thigh_length}"/></geometry>
+        <geometry><cylinder radius="${0.014 * scale}" length="${thigh_length}"/></geometry>
       </collision>
-      <xacro:cylinder_inertia mass="${thigh_mass}" radius="0.014" length="${thigh_length}"/>
+      <xacro:cylinder_inertia mass="${thigh_mass}" radius="${0.014 * scale}" length="${thigh_length}"/>
     </link>
     <!-- calf: knee pitch. The foot pad is a sphere on this link rather than a
@@ -66,5 +66,5 @@
       <visual>
         <origin xyz="0 0 ${-calf_length / 2.0}" rpy="0 0 0"/>
-        <geometry><cylinder radius="0.011" length="${calf_length}"/></geometry>
+        <geometry><cylinder radius="${0.011 * scale}" length="${calf_length}"/></geometry>
         <material name="cat_fur"/>
       </visual>
@@ -80,5 +80,5 @@
         <geometry><sphere radius="${foot_radius}"/></geometry>
       </collision>
-      <xacro:cylinder_inertia mass="${calf_mass}" radius="0.011" length="${calf_length}"/>
+      <xacro:cylinder_inertia mass="${calf_mass}" radius="${0.011 * scale}" length="${calf_length}"/>
     </link>
     <!-- Reference frame at the contact point, for debugging in RViz/tf. -->
