Commit message: Separate construction weight from size, and find what the torque really is
mass_scale is a second knob alongside scale. scale^3 assumes the animal is
solid with whatever the 3.7 kg original was made of, which turns a 22 cm cat
into a 24 kg robot at scale 1.87; mass_scale 0.62 models a hollow frame at the
same dimensions, about what Unitree's Go2 weighs for its size.

It was added to answer "will a lighter build need smaller actuators", and the
answer turned out to be no - which is the useful part.

Measured at 50 cm walking 0.1 m/s, worst joint, 95th percentile:

    24.2 kg   28.6 Nm
    15.0 kg   27.2 Nm

A 38% mass cut bought 5%. Speed does not help either (0.94 m/s and 0.1 m/s
land within noise of each other), nor duty factor (0.65 vs 0.50: 26.4 vs
26.0), nor swing height. Three plausible mechanisms tested and disproved:
footfall impact, knee-dominated loading, and stance over-constraint.

What it actually is, from the one measurement that did scale:

    standing, 24.2 kg   8.4 Nm
    standing, 15.0 kg   5.2 Nm   (predicted 5.21 - gravity, exactly linear)
    walking, median     1-2 Nm
    walking, 95th pct   27 Nm

Standing scales with mass perfectly, so the effort readings are physical. The
~22 Nm that walking adds on top does not scale with anything, because it is
not gravity: the gait is open loop, the body does not follow the plan exactly,
and a planted foot is commanded to a place it is not - so the position
controller leans on the ground until friction or the effort limit stops it.
That force depends on tracking error, not on what the robot weighs.

This matters for actuator choice: sizing to the 95th percentile sizes for a
control artifact. The physical requirement for a slow walk is much closer to
the standing figure. The fix is compliance or feedback, not bigger motors -
which is an argument for the IMU work, not against the cheap actuators.

Co-Authored-By: Claude Opus 5 <noreply@anthropic.com>

File: src/robot_cat_description/urdf/cat.urdf.xacro (robot description, xacro)
@@ -17,4 +17,13 @@
   <xacro:arg name="scale" default="1.0"/>
   <xacro:property name="scale" value="$(arg scale)"/>
+  <!-- Construction weight, separate from size. scale^3 assumes the animal is
+       filled with whatever the 3.7 kg original was made of, which is how a
+       22 cm cat becomes a 24 kg robot at scale 1.87. A real build is hollow:
+       Unitree's Go2 is 15 kg at about that size, so mass_scale 0.62 models a
+       lightweight frame at the same dimensions. Torque tracks mass almost
+       linearly in a quasi-static walk, so this is the cheapest lever there
+       is on actuator class - cheaper than shrinking the robot. -->
+  <xacro:arg name="mass_scale" default="1.0"/>
+  <xacro:property name="mass_scale" value="$(arg mass_scale)"/>
   <!-- ==================== dimensions ====================
        These MUST match LegGeometry in robot_cat_gait/leg_ik.py. If you change
@@ -53,16 +62,16 @@
        So they carry token mass, damped enough to settle rather than swing,
        and `body_mass` carries what they gave up - total mass is unchanged. -->
-  <xacro:property name="body_mass"  value="${2.23 * scale**3}"/>
-  <xacro:property name="head_mass"  value="${0.06 * scale**3}"/>
-  <xacro:property name="neck_mass"  value="${0.01 * scale**3}"/>
-  <xacro:property name="tail_mass"  value="${0.015 * scale**3}"/>
+  <xacro:property name="body_mass"  value="${2.23 * scale**3 * mass_scale}"/>
+  <xacro:property name="head_mass"  value="${0.06 * scale**3 * mass_scale}"/>
+  <xacro:property name="neck_mass"  value="${0.01 * scale**3 * mass_scale}"/>
+  <xacro:property name="tail_mass"  value="${0.015 * scale**3 * mass_scale}"/>
   <!-- Cosmetic joints only. Far stiffer than the legs: they are meant to hold
        a pose, and any wobble here feeds straight back into the trunk. -->
   <xacro:property name="trim_damping" value="0.4"/>
-  <xacro:property name="hip_mass"   value="${0.10 * scale**3}"/>
+  <xacro:property name="hip_mass"   value="${0.10 * scale**3 * mass_scale}"/>
   <!-- Scaled with the 0.09 -> 0.11 lengthening, so the longer links do not
        quietly become less dense than the ones they replaced. -->
-  <xacro:property name="thigh_mass" value="${0.147 * scale**3}"/>
-  <xacro:property name="calf_mass"  value="${0.098 * scale**3}"/>
+  <xacro:property name="thigh_mass" value="${0.147 * scale**3 * mass_scale}"/>
+  <xacro:property name="calf_mass"  value="${0.098 * scale**3 * mass_scale}"/>
   <!-- ==================== joint properties ====================
        Ranges are deliberately generous for the pitch joints so the gait has

Commit message: Put the real ST3215 and the real masses into the model
The simulation declared 20 Nm and 20 rad/s in every joint - placeholder
numbers matching no actuator that can be bought - and carried 3.7 kg of
scaled cat density rather than a parts list. Both are now the hardware:
2.57 Nm, which is the ST3215 stall torque at the worst state of a 3S pack,
and 4.7 rad/s no-load. Head and tail get a microservo's 0.20 Nm instead of
a leg servo's.

Masses become the purchase plan, 2.095 kg, distributed by where the parts
physically sit. The roll servo bolts to the trunk so its mass is the
trunk's; hip_link carries the thigh servo it swings, thigh_link the knee
servo, and calf_link is unpowered. That leaves the swing leg light, which
is what it wants to be.

Torque figures in the documents are scaled linearly from the measured run
at 2.03 kg and labelled as such - the redistribution shifts mass between
links, so one Gazebo run still owes a confirmation. It is listed as an
open item rather than quietly presented as measured.

Also fixes the withers figure, which read 21.7 cm in the model comment
against 24.2 cm everywhere else. 24.2 is right: hip 17.2 plus half the
trunk depth.

Compute moves to Raspberry Pi 5 with the AI HAT+. The Pi 4B has no PCIe
connector, so the Hailo accelerator is impossible with it rather than
slower, and object recognition is the thing the vision plan is built on.
That decision costs the budget: the list comes to 3788.60 zl against the
2500 it started from, and the whole difference is this one line. It is
stated plainly at the top of the plan rather than buried. Three
consequences travel with it and are now documented - the Active Cooler is
not optional under a HAT, the camera needs a 22-pin cable the module does
not ship with, and a Pi 5 with an accelerator wants most of what the
D24V50F5 can give, so the microservos and audio get a converter of their
own.

The assembly document gains what the parts list never had: mounts. Pi
standoffs at the 58 x 49 mm M2.5 pattern, standoffs for every module,
a strap for a battery that must not be glued because it swells, bearings
for the passive side of all twelve joints, enough threaded inserts for a
whole cat rather than one leg, cable grommets, and paw pads - which the
document already argued were load-bearing without ever putting them on a
list to buy.

Documents now carry only current values. The STS3250 verdict, computed for
a 3.7 kg robot and already withdrawn by the actuator report, is gone from
the electronics notes along with the section describing the fictional
motors this commit removed. The purchase plan collapses from two variants
plus a camera comparison to one list. The scale chart went with them: both
its anchor points were measured at masses that no longer exist, and a
chart that cannot be re-measured here is worse than no chart.

Two fixes found on the way. The DejaVu lookup picked a directory from
DejaVuSans.ttf and assumed the oblique sat beside it, which is false on
Debian's fonts-dejavu-core, so both scripts using it crashed on a stock
Ubuntu; each face now resolves on its own with the matplotlib fallback.
And the report README says what these documents are for: current state, no
change history.

Co-Authored-By: Claude Opus 5 <noreply@anthropic.com>
Claude-Session: https://claude.ai/code/session_01GBkNLAG8VG58owhw5DdrBF

File: src/robot_cat_description/urdf/cat.urdf.xacro (robot description, xacro)
@@ -10,27 +10,22 @@
        multiplied by this; masses go as scale^3 and joint effort as scale^4,
        which is how joint torque actually scales (mass x lever arm).
-       1.00 is a real domestic cat and is the right default: 24.2 cm at the
-       withers against a live cat's 24, and 3.7 kg against 3.6-5.4. Nothing
-       needs multiplying to get there. (An earlier revision briefly defaulted
-       to 1.11 on the strength of a stale 21.7 cm figure, taken before the
-       chest was deepened to cat proportions; deepening the body raised the
-       withers, and 1.11 then overshot to 26.9 cm.)
-       Scale is not a cosmetic choice, it picks an actuator class. Measured
-       walking at 0.1 m/s, worst joint, 95th percentile:
-           1.00 (real cat, 3.7 kg)    ~5 Nm
-           1.87 (50 cm, 24 kg)        27 Nm
-       Torque goes as roughly the 3.5 power of size, so a robot that merely
-       looks bigger costs five times the motor. 1.87 is what "about 50 cm
-       tall" works out to if the animal keeps cat proportions - and at that
-       size a cat-shaped thing is a lynx, which really does weigh 20 kg. -->
+       1.00 is the robot that gets built: 24.2 cm at the withers against a
+       live cat's 24, and 2.1 kg of servos, printed shell, battery and
+       electronics. Nothing needs multiplying to get there, and the ST3215
+       torque limit below is only true at this scale.
+       Scale is not a cosmetic choice, it picks an actuator class. Torque
+       goes as roughly the 3.5 power of size, so an animal that merely looks
+       bigger costs several times the motor and leaves the ST3215 class
+       entirely. Anything other than 1.00 needs its own torque measurement
+       before it means anything. -->
   <xacro:arg name="scale" default="1.0"/>
   <xacro:property name="scale" value="$(arg scale)"/>
-  <!-- Construction weight, separate from size. scale^3 assumes the animal is
-       filled with whatever the 3.7 kg original was made of, which is how a
-       22 cm cat becomes a 24 kg robot at scale 1.87. A real build is hollow:
-       Unitree's Go2 is 15 kg at about that size, so mass_scale 0.62 models a
-       lightweight frame at the same dimensions. Torque tracks mass almost
-       linearly in a quasi-static walk, so this is the cheapest lever there
-       is on actuator class - cheaper than shrinking the robot. -->
+  <!-- Construction weight, separate from size. The masses below are the
+       parts list, so 1.0 is the robot as specified and needs no correction.
+       The knob exists to ask what a heavier or lighter build would cost in
+       torque: it tracks mass almost linearly in a quasi-static walk, which
+       makes it the cheapest lever there is on actuator class. The obvious
+       use is checking the PETG estimate - the shell is 700 g of the 2.1 kg
+       and is the one figure nobody has weighed yet. -->
   <xacro:arg name="mass_scale" default="1.0"/>
   <xacro:property name="mass_scale" value="$(arg mass_scale)"/>
@@ -40,10 +35,10 @@
        places the legs cannot reach. -->
   <xacro:property name="hip_offset"   value="${0.025 * scale}"/>  <!-- hip roll -> thigh pitch, lateral -->
-  <!-- 0.09 made a long, low animal: 18.7 cm at the withers over a 22 cm hip
-       span, a ratio of 0.85. A cat is close to square in profile - it stands
-       about as tall at the shoulder as its trunk is long - so the old figure
-       read as a dachshund. 0.11 puts the withers at 21.7 cm for a ratio of
-       0.99, and holds the standing knee at the same 73% of full reach the
-       0.09 leg had, so the gait keeps its bend and its swing clearance. -->
+  <!-- A cat is close to square in profile - it stands about as tall at the
+       shoulder as its trunk is long. 0.11 puts the hip 17.2 cm up and the
+       withers at 24.2 cm over a 22 cm hip span, and holds the standing knee
+       at 73% of full reach, which is what gives the gait its bend and its
+       swing clearance. Segment length and stance_height move together:
+       raising one alone straightens the knee towards a locked leg. -->
   <xacro:property name="thigh_length" value="${0.11 * scale}"/>   <!-- L1 -->
   <xacro:property name="calf_length"  value="${0.11 * scale}"/>   <!-- L2 -->
@@ -51,6 +46,6 @@
   <!-- A cat's trunk is deeper than it is wide - chest girth of about
        38 cm works out near 14 cm deep by 10 cm across - so the box is
-       length : width : depth = 1 : 0.37 : 0.47. The old 1 : 0.47 : 0.30 was
-       the other way round and read as a slab on legs rather than an animal. -->
+       length : width : depth = 1 : 0.37 : 0.47. Keep it that way round: a
+       trunk wider than it is deep reads as a slab on legs, not an animal. -->
   <xacro:property name="body_length" value="${0.30 * scale}"/>
   <xacro:property name="body_width"  value="${0.111 * scale}"/>
@@ -60,27 +55,39 @@
   <xacro:property name="hip_y" value="${0.055 * scale}"/>
   <!-- ==================== masses ====================
-       The head and tail are cosmetic but no longer fixed joints, so their
-       mass is a free body hanging off the trunk instead of being lumped into
-       it by SDF conversion. Two things follow, and both showed up as a
-       visibly bouncier trot when the tail was actuated:
-       * the trunk lost the parallel-axis share those masses used to
-         contribute to its pitch inertia (0.0263 -> 0.0164, a 38% drop), so
-         it now pitches far more readily each half stride;
-       * whatever mass they keep slops about on a long lever at the very
-         ends of the body, exactly where it disturbs pitch most.
-       So they carry token mass, damped enough to settle rather than swing,
-       and `body_mass` carries what they gave up - total mass is unchanged. -->
-  <xacro:property name="body_mass"  value="${2.23 * scale**3 * mass_scale}"/>
-  <xacro:property name="head_mass"  value="${0.06 * scale**3 * mass_scale}"/>
-  <xacro:property name="neck_mass"  value="${0.01 * scale**3 * mass_scale}"/>
-  <xacro:property name="tail_mass"  value="${0.015 * scale**3 * mass_scale}"/>
-  <!-- Cosmetic joints only. Far stiffer than the legs: they are meant to hold
-       a pose, and any wobble here feeds straight back into the trunk. -->
-  <xacro:property name="trim_damping" value="0.4"/>
-  <xacro:property name="hip_mass"   value="${0.10 * scale**3 * mass_scale}"/>
-  <!-- Scaled with the 0.09 -> 0.11 lengthening, so the longer links do not
-       quietly become less dense than the ones they replaced. -->
-  <xacro:property name="thigh_mass" value="${0.147 * scale**3 * mass_scale}"/>
-  <xacro:property name="calf_mass"  value="${0.098 * scale**3 * mass_scale}"/>
+       These are the parts list, not a scaled animal, and they sum to the
+       2.095 kg budget in docs/napedy-v4.pdf. Where each part physically
+       sits decides which link carries it, and the servos dominate: twelve
+       ST3215 at 69 g are 828 g of the total.
+       The roll servo is bolted to the trunk, so its mass is base_link's.
+       hip_link carries the thigh pitch servo it swings, thigh_link carries
+       the knee servo at the knee, and calf_link is unpowered - printed
+       segment, paw pad and the wiring crossing it. That makes the lower leg
+       light, which is what a swing leg wants.
+           base_link  1042 g   4 roll servos, battery, Pi 5 + AI HAT+,
+                               trunk shell, converters, wiring
+           head         80 g   shell, camera, IR illuminator, 2 microservos
+           tail         27 g   shell and its microservo
+           per leg     234 g   88 hip + 109 thigh + 37 calf
+       Head and tail are actuated, not fixed, so their mass hangs off the
+       trunk on a long lever instead of being lumped into it by SDF
+       conversion - exactly where it disturbs pitch most. They are damped
+       stiffly below so they settle rather than swing. -->
+  <xacro:property name="body_mass"  value="${1.042 * scale**3 * mass_scale}"/>
+  <xacro:property name="head_mass"  value="${0.080 * scale**3 * mass_scale}"/>
+  <xacro:property name="neck_mass"  value="${0.010 * scale**3 * mass_scale}"/>
+  <xacro:property name="tail_mass"  value="${0.027 * scale**3 * mass_scale}"/>
+  <xacro:property name="hip_mass"   value="${0.088 * scale**3 * mass_scale}"/>
+  <xacro:property name="thigh_mass" value="${0.109 * scale**3 * mass_scale}"/>
+  <xacro:property name="calf_mass"  value="${0.037 * scale**3 * mass_scale}"/>
+  <!-- Head and tail joints. Damped far stiffer than the legs: they are meant
+       to hold a pose, and any wobble here feeds straight back into the trunk.
+       Effort and velocity are a metal-gear microservo of the class the parts
+       list budgets for - the plan names three of them but not a model, so
+       0.20 Nm is the conservative end of that class rather than a datasheet
+       figure. It is ample either way: the head is 80 g on a 3 cm lever, so
+       holding it up takes 0.024 Nm. -->
+  <xacro:property name="trim_damping"  value="0.4"/>
+  <xacro:property name="trim_effort"   value="${0.20 * scale**4}"/>
+  <xacro:property name="trim_velocity" value="8.0"/>
   <!-- ==================== joint properties ====================
        Ranges are deliberately generous for the pitch joints so the gait has
@@ -92,6 +99,21 @@
   <xacro:property name="calf_lower"     value="-2.70"/>
   <xacro:property name="calf_upper"     value="-0.10"/>
-  <xacro:property name="joint_effort"   value="${20.0 * scale**4}"/>
-  <xacro:property name="joint_velocity" value="20.0"/>
+  <!-- The actuator is a Waveshare ST3215, and these are its numbers, not
+       headroom picked to make the simulation behave.
+       Effort is stall torque at the *worst* battery state. The datasheet
+       30 kg.cm is quoted at 12 V and a DC motor's stall torque tracks
+       voltage, so a 3S pack gives 3.08 Nm freshly charged and 2.57 Nm by the
+       time it is nearly flat. Sizing on 2.57 means the cat does not get
+       weaker than the simulation as the battery drains. The walk needs
+       1.93 Nm at the 95th percentile, so this is about 33% margin.
+       Velocity is the no-load figure, 0.222 s/60 degrees at 12 V. The gait
+       peaks near 2.8 rad/s, so it fits, but not by so much that a faster
+       cycle time is free.
+       Effort keeps the scale^4 factor because required torque scales that
+       way; the ST3215 itself does not, so any scale but 1.00 has left this
+       actuator behind. Velocity is unscaled - a servo turns at the speed it
+       turns regardless of how big the animal around it is. -->
+  <xacro:property name="joint_effort"   value="${2.57 * scale**4}"/>
+  <xacro:property name="joint_velocity" value="4.7"/>
   <xacro:property name="joint_damping"  value="0.05"/>
   <xacro:property name="joint_friction" value="0.01"/>
@@ -126,5 +148,5 @@
     <origin xyz="${body_length/2} 0 ${body_height/2}" rpy="0 0 0"/>
     <axis xyz="0 0 1"/>
-    <limit lower="-0.6" upper="0.6" effort="5" velocity="6"/>
+    <limit lower="-0.6" upper="0.6" effort="${trim_effort}" velocity="${trim_velocity}"/>
     <dynamics damping="${trim_damping}" friction="${joint_friction}"/>
   </joint>
@@ -141,5 +163,5 @@
          convention below and by robot_cat_teleop. -->
     <axis xyz="0 -1 0"/>
-    <limit lower="-0.3" upper="0.5" effort="5" velocity="6"/>
+    <limit lower="-0.3" upper="0.5" effort="${trim_effort}" velocity="${trim_velocity}"/>
     <dynamics damping="${trim_damping}" friction="${joint_friction}"/>
   </joint>
@@ -159,7 +181,8 @@
          Only one of them is a camera. Stereo exists solely to recover depth,
          and docs/plan-zakupowy.pdf takes depth from a VL53L5CX time-of-flight
-         sensor instead - two camera modules would need syncing and
-         calibrating on a machine that shakes as it walks, and a Pi 4B has a
-         single CSI port anyway.
+         sensor instead: two camera modules would need syncing and calibrating
+         on a machine that shakes as it walks, and the other socket is spoken
+         for by the illuminator. The Pi 5 does have two CSI ports, so stereo
+         stays physically possible - it is just not what the depth comes from.
          The camera is the *NoIR* variant - no infrared cut filter, so it sees
          the illuminator and the cat can see in the dark. That costs correct
@@ -213,5 +236,5 @@
     <!-- Wider than the sweep TailParams actually uses, so the controller
          settles on its target instead of pushing against the joint stop. -->
-    <limit lower="-1.4" upper="1.0" effort="5" velocity="6"/>
+    <limit lower="-1.4" upper="1.0" effort="${trim_effort}" velocity="${trim_velocity}"/>
     <dynamics damping="${trim_damping}" friction="${joint_friction}"/>
   </joint>
